File: PCB/Joy Board.kicad_sch (KiCad schematic)
At the start: 134 parts, among them SW1 SW_Push, SW10 SW_Push, SW11 SW_Push, SW12 SW_Push, SW13 SW_Push, SW14 SW_Push, SW15 SW_Push, SW16 SW_Push, SW17 SW_Push, SW18 SW_Push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

Commit message: firmware done and updated to latest pcb
Parts:
- R10, R12, R13, R15: value 1k -> 10k
- R11, R14, R16, R9: value 2k -> 22k
- R5, R6, R7, R8: value 200 -> 2.4k
Changed lines of the file:
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@@
 			)
 		)
-		(property "Value" "200"
+		(property "Value" "2.4k"
 			(at 95.25 175.26 90)
 			(effects
@@
 			)
 		)
-		(property "Value" "2k"
+		(property "Value" "22k"
 			(at 82.55 173.9899 0)
 			(effects
@@
 			)
 		)
-		(property "Value" "200"
+		(property "Value" "2.4k"
 			(at 154.94 207.01 90)
 			(effects
@@
 			)
 		)
-		(property "Value" "1k"
+		(property "Value" "10k"
 			(at 72.39 222.2499 0)
 			(effects
@@
 			)
 		)
-		(property "Value" "1k"
+		(property "Value" "10k"
 			(at 132.08 196.85 90)
 			(effects
@@
 			)
 		)
-		(property "Value" "200"
+		(property "Value" "2.4k"
 			(at 53.34 198.12 90)
 			(effects
@@
 			)
 		)
-		(property "Value" "1k"
+		(property "Value" "10k"
 			(at 72.39 165.1 90)
 			(effects
@@
 			)
 		)
-		(property "Value" "1k"
+		(property "Value" "10k"
 			(at 40.64 198.1199 0)
 			(effects
@@
 			)
 		)
-		(property "Value" "2k"
+		(property "Value" "22k"
 			(at 62.23 213.36 90)
 			(effects
@@
 			)
 		)
-		(property "Value" "2k"
+		(property "Value" "22k"
 			(at 142.24 205.7399 0)
 			(effects
@@
 			)
 		)
-		(property "Value" "2k"
+		(property "Value" "22k"
 			(at 30.48 189.23 90)
 			(effects
@@
 			)
 		)
-		(property "Value" "200"
+		(property "Value" "2.4k"
 			(at 85.09 226.06 90)
 			(effects
