File: PCB/Joy Board.kicad_pcb (KiCad board)
At the start: 2 copper layers, 282.6 x 138.1 mm, 132 parts, among them SW1 SW_Push, SW10 SW_Push, SW11 SW_Push, SW12 SW_Push, SW13 SW_Push, SW14 SW_Push, SW15 SW_Push, SW16 SW_Push, SW17 SW_Push, SW18 SW_Push, SW19 SW_Push, SW2 SW_Push, SW20 SW_Push, SW3 SW_Push, SW4 SW_Push, SW5 SW_Push, SW6 SW_Push, SW7 SW_Push, SW8 SW_Push, SW9 SW_Push, U1 SuperMini nRF52840, U2 SuperMini nRF52840, U3 COM-09032

Commit message: different pcbs
Parts:
- removed H1, H2, H3: MountingHole, mouse_bit:mouse-bite-5mm-slot
Other:
- outline, holes or cut-outs redrawn
